File: hw/lse1_pcb/lse1_pcb.kicad_pcb (KiCad board)
At the start: 4 copper layers, 100 x 100 mm, 74 parts, among them J1 PWR_IN, J2 DataOut, M1 Motor_3pin, Q1 IRFR1205, Q2 IRFR1205, Q3 IRFR1205, Q4 IRFR1205, Q5 IRFR1205, Q6 IRFR1205, U1 IR2301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

Commit message: difference describe/commit?
Parts:
- added U6: EK-TM4C123GXL, models:MODULE_EK-TM4C123GXL, F.Cu at (112.1, 112.2)

Commit message: ponts fets
Parts:
- removed J2: DataOut, Connector_PinHeader_2.54mm:PinHeader_2x06_P2.54mm_Vertical
- added J3: DataOut, Connector_PinHeader_2.54mm:PinHeader_2x06_P2.54mm_Vertical, F.Cu at (162.4, 108.2)
- added U4: AZ1084CD-5.0TRG1, models_cachy:DPAK457P1010X238-3N, F.Cu at (191.2, 102.9)
- CBOOT1, CBOOT2, CBOOT3: moved to B.Cu
- moved Cd2 147.1 mm to (23.7, 61.8)
- moved Cdec6 147.1 mm to (35.0, 48.4)
- moved Cdec7 147.1 mm to (35.0, 51.7)
- moved Cfilt1 147.1 mm to (35.0, 55.1)
- moved Cfilt3 147.1 mm to (35.0, 61.8)
- moved D6 147.1 mm to (45.5, 64.8)
- moved R18 147.1 mm to (34.9, 25.2)
- moved R19 147.1 mm to (34.9, 28.5)
- moved R20 147.1 mm to (34.9, 31.8)
- moved R21 147.1 mm to (34.9, 35.1)
- moved Rled5 147.1 mm to (34.9, 45.0)
- moved Rled_dbg0 147.1 mm to (40.5, 25.2)
- moved Rpull0 147.1 mm to (40.5, 28.5)
- moved Rpull1 147.1 mm to (40.5, 31.8)
- moved Rpull2 147.1 mm to (40.5, 35.1)
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Routing:
- net FASE2: track 0.00 -> 16.7 mm, vias 0 -> 15
- net +3.3V: track 0.00 -> 10.7 mm
- net FASE1: track 0.00 -> 6.98 mm, vias 0 -> 15
- net FASE3: track 0.00 -> 6.92 mm, vias 0 -> 15
- net /BOOT3: track 0.00 -> 4.91 mm
- net /BOOT2: track 0.00 -> 4.83 mm
- net /BOOT1: track 0.00 -> 4.74 mm
- net /PWRLED: track 0.00 -> 4.22 mm
- net Net-(Q1-G): track 0.00 -> 2.78 mm
- net /HO1: track 0.00 -> 2.76 mm
- net /HO2: track 0.00 -> 2.73 mm
- net Net-(Q5-G): track 0.00 -> 2.72 mm
- net /HO3: track 0.00 -> 2.72 mm
- net Net-(Q3-G): track 0.00 -> 2.64 mm
- net Net-(Q2-G): track 0.00 -> 2.46 mm
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- added copper zone on F.Cu, net +12V
- added copper zone on In1.Cu, net +12V
- added copper zone on F.Cu, net +5V
- added copper zone on B.Cu, net FASE1
- added copper zone on F.Cu, net FASE1
- added copper zone on B.Cu, net FASE2
- added copper zone on F.Cu, net FASE2
- added copper zone on B.Cu, net FASE3
- added copper zone on F.Cu, net FASE3
- added copper zone on F.Cu, net GND
- added copper zone on In2.Cu, net GND
Other:
- board size 100 x 100 mm -> 73.9 x 107.2 mm
- board text added: "D1"

Commit message: pcb done
Parts:
- removed TP4, TP5, TP6: TestPoint, Connector_PinHeader_2.54mm:PinHeader_1x01_P2.54mm_Vertical
- Cfilt1, Cfilt2, Cfilt3, R13, R14, R15, R16, R17: moved to B.Cu
- moved Rled_dbg0 206.4 mm to (227.6, 112.3), turned to 90 degrees
- moved Cd3 197.9 mm to (221.5, 67.7), turned to 180 degrees
- moved R23 188.9 mm to (221.2, 73.1)
- moved Cdec6 187.8 mm to (221.5, 70.0), turned to 180 degrees
- moved D6 187.1 mm to (227.6, 108.2), turned to 90 degrees
- moved R22 185.9 mm to (217.8, 72.0), turned to -90 degrees
- moved TP1 184.3 mm to (227.6, 84.4)
- moved TP2 184.3 mm to (227.6, 89.0)
- moved TP3 184.3 mm to (227.6, 93.6)
- moved TP7 181.8 mm to (227.7, 98.4)
- moved Cd2 181.6 mm to (205.2, 67.7), turned to 180 degrees
- moved R17 181.1 mm to (201.1, 93.7), turned to -90 degrees
- moved R15 180.7 mm to (204.5, 86.0), turned to 180 degrees
- moved R14 177.7 mm to (201.1, 83.7), turned to -90 degrees
- moved R16 177.2 mm to (201.1, 88.2), turned to -90 degrees
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Connections:
- net Net-(R13-Pad1) renamed /STAR
- Cfilt1 pad 1: Net-(U5A-+) -> Net-(U5B-+)
- Cfilt2 pad 1: Net-(U5B-+) -> Net-(U5A-+)
- R18 pad 2: Net-(U5A-+) -> Net-(U5B-+)
- R19 pad 1: Net-(U5A-+) -> Net-(U5B-+)
- R20 pad 2: Net-(U5B-+) -> Net-(U5A-+)
- R21 pad 1: Net-(U5B-+) -> Net-(U5A-+)
- U5 pad 1: MEAS2 -> MEAS1
- U5 pad 2: MEAS1 -> MEAS2
- U6 pad J1_3: MEAS1 -> unconnected-(U6-PB0-PadJ1_3)
- U6 pad J1_4: MEAS2 -> unconnected-(U6-PB1-PadJ1_4)
- U6 pad J2_10: unconnected-(U6-PA2-PadJ2_10) -> Net-(D6-A)
- U6 pad J2_2: MEAS3 -> unconnected-(U6-PB2-PadJ2_2)
- U6 pad J4_1: unconnected-(U6-PF2-PadJ4_1) -> MEAS1
- U6 pad J4_4: unconnected-(U6-PC4-PadJ4_4) -> MEAS2
- U6 pad J4_5: Net-(D6-A) -> unconnected-(U6-PC5-PadJ4_5)
- U6 pad J4_6: unconnected-(U6-PC6-PadJ4_6) -> MEAS3
Routing:
- net PWM3B: track 0.00 -> 75.1 mm, vias 0 -> 1
- net PWM3A: track 0.00 -> 67.4 mm, vias 0 -> 1
- net NEUT: track 0.00 -> 47.8 mm
- net PWM2B: track 0.00 -> 46.3 mm, vias 0 -> 1
- net Net-(U5C-+): track 0.00 -> 39.8 mm, vias 0 -> 1
- net PWM2A: track 0.00 -> 37.6 mm, vias 0 -> 1
- net +5V: track 0.00 -> 34.5 mm
- net MEAS1: track 0.00 -> 34.0 mm, vias 0 -> 1
- net MEAS3: track 0.00 -> 33.8 mm, vias 0 -> 1
- net MEAS2: track 0.00 -> 32.9 mm, vias 0 -> 1
- net PWM1B: track 0.00 -> 31.4 mm, vias 0 -> 1
- net FASE1: track 6.98 -> 38.2 mm, vias 15 -> 9
- net +3.3V: track 10.7 -> 38.7 mm, vias 0 -> 9
- net FASE3: track 6.92 -> 34.2 mm, vias 15 -> 9
- net Net-(U6-~{TARGETRST}): track 0.00 -> 26.8 mm
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- added copper zone on F.Cu, net +3.3V
- added copper zone on In2.Cu, net +3.3V
- added copper zone on B.Cu, net /STAR
- added copper zone on B.Cu, net NEUT
- added copper zone on F.Cu, net NEUT
Other:
- board size 73.9 x 107.2 mm -> 65 x 94.6 mm

Commit message: copper pours i algunes modificacions
Routing:
- added copper zone on B.Cu, net GND
Changed lines of the file:
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@@
 		(tags "capacitor electrolytic nonpolar")
 		(property "Reference" "CPWR0"
-			(at 0 -6.2 90)
+			(at -0.155 0.075 180)
 			(layer "F.SilkS")
 			(effects
@@
 		(tags "resistor")
 		(property "Reference" "Rled12"
-			(at 0 -1.83 0)
+			(at 0.075 0.03 0)
 			(layer "F.SilkS")
+			(hide yes)
 			(effects
 				(font
@@
 		(tags "LED")
 		(property "Reference" "D4"
-			(at 0 -1.65 0)
+			(at 0.065 0.07 0)
 			(layer "F.SilkS")
 			(effects
@@
 			(at 0.6625 -1.9 90)
 			(layer "F.SilkS")
+			(hide yes)
 			(effects
 				(font
@@
 		(tags "Through hole pin header THT 1x01 2.54mm single row")
 		(property "Reference" "TP7"
-			(at 0.1 -1.3 0)
+			(at 0.01 -2.33 0)
 			(layer "F.SilkS")
 			(effects
@@
 		(tags "resistor")
 		(property "Reference" "R13"
-			(at 0 0 90)
+			(at 0 1.835 180)
 			(layer "B.SilkS")
 			(effects
@@
 		(tags "resistor")
 		(property "Reference" "R16"
-			(at 0 0 0)
+			(at 0 -2.78 0)
 			(layer "B.SilkS")
 			(effects
@@
 		(tags "resistor")
 		(property "Reference" "R15"
-			(at -1.75 0.01 90)
+			(at -0.4775 1.725 180)
 			(layer "B.SilkS")
 			(effects
@@
 		(tags "resistor")
 		(property "Reference" "R14"
-			(at 0 0 0)
+			(at -2.9975 0 0)
 			(layer "B.SilkS")
 			(effects
@@
 		(layer "F.Cu")
 		(hatch edge 0.5)
+		(priority 1)
+		(connect_pads yes
+			(clearance 0.5)
+		)
+		(min_thickness 0.25)
+		(filled_areas_thickness no)
+		(fill yes
+			(thermal_gap 0.5)
+			(thermal_bridge_width 0.5)
+		)
+		(polygon
+			(pts
+				(xy 153.1 39.63) (xy 242.68 39.63) (xy 244.16 143.27) (xy 152.31 141.57)
+			)
+		)
+	)
+	(zone
+		(net 4)
+		(net_name "GND")
+		(layer "F.Cu")
+		(hatch edge 0.5)
 		(priority 99)
 		(connect_pads
@@
 			)
 		)
+	)
+	(zone
+		(net 4)
+		(net_name "GND")
+		(layer "B.Cu")
+		(hatch edge 0.5)
+		(priority 1)
+		(connect_pads yes
+			(clearance 0.5)
+		)
+		(min_thickness 0.25)
+		(filled_areas_thickness no)
+		(fill yes
+			(thermal_gap 0.5)
+			(thermal_bridge_width 0.5)
+		)
+		(polygon
+			(pts
+				(xy 149.58 38.83) (xy 247.67 38.72) (xy 247.9 148.72) (xy 149.47 143.5)
+			)
+		)
