File: hw/lse1_pcb/lse1_pcb.kicad_pcb (KiCad board)
At the start: 4 copper layers, 65 x 94.6 mm, 73 parts, among them J1 PWR_IN, J3 DataOut, M1 Motor_3pin, Q1 IRFR1205, Q2 IRFR1205, Q3 IRFR1205, Q4 IRFR1205, Q5 IRFR1205, Q6 IRFR1205, U1 IR2301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

Commit message: restore backup, design up-to-date
Parts:
- Cdec7, Rpull1, Rpull2, Rpull3, U5: moved to B.Cu
- moved J3 63.4 mm to (230.0, 104.8), turned to 180 degrees
- moved TP1 60.5 mm to (171.6, 107.3), turned to 180 degrees
- moved D6 60.2 mm to (171.9, 85.4)
- moved Rled_dbg0 60.2 mm to (171.9, 89.5)
- moved Rled5 58.4 mm to (237.9, 137.2), turned to 90 degrees
- moved TP7 57.8 mm to (171.5, 112.1), turned to 180 degrees
- moved TP2 57.7 mm to (171.6, 102.7), turned to 180 degrees
- moved TP3 56.2 mm to (171.6, 98.1), turned to 180 degrees
- moved Rpull0 56.0 mm to (232.2, 141.0), turned to 0 degrees
- moved Cdec3 54.7 mm to (222.5, 110.9), turned to -90 degrees
- moved Cdec2 43.4 mm to (218.4, 111.7), turned to 0 degrees
- moved CPWR0 35.5 mm to (241.6, 152.2)
- moved D4 35.5 mm to (234.3, 154.2)
- moved J1 35.5 mm to (252.1, 149.7)
- moved Rled12 35.5 mm to (233.8, 150.4)
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Routing:
- net PWM3B: track 75.1 -> 18.3 mm, vias 1 -> 0
- net PWM3A: track 67.4 -> 14.7 mm, vias 1 -> 0
- net +3.3V: track 38.7 -> 2.10 mm, vias 9 -> 40
- net NEUT: track 47.8 -> 16.1 mm
- net PWM2B: track 46.3 -> 15.4 mm, vias 1 -> 0
- net PWM2A: track 37.6 -> 10.2 mm, vias 1 -> 0
- net Net-(U6-~{TARGETRST}): track 26.8 -> 0.00 mm
- net Net-(U5A-+): track 21.0 -> 43.3 mm
- net MEAS1: track 34.0 -> 12.5 mm, vias 1 -> 0
- net PWM1B: track 31.4 -> 11.9 mm, vias 1 -> 0
- net MEAS3: track 33.8 -> 15.3 mm, vias 1 -> 0
- net MEAS2: track 32.9 -> 15.4 mm, vias 1 -> 0
- net Net-(U5C-+): track 39.8 -> 25.5 mm, vias 1 -> 2
- net Net-(U5B-+): track 23.5 -> 10.4 mm, vias 1 -> 2
- net PWM1A: track 14.8 -> 5.05 mm, vias 1 -> 0
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- added copper zone on B.Cu, net +3.3V
- removed copper zone on F.Cu, net +3.3V
- removed copper zone on F.Cu, net NEUT
Other:
- board size 65 x 94.6 mm -> 67.4 x 94.6 mm

Commit message: close to finish
Parts:
- Rpull0: moved to B.Cu
- moved J1 84.0 mm to (170.1, 131.4), turned to 180 degrees
- moved CPWR0 65.3 mm to (180.6, 128.9), turned to -90 degrees
- moved Rpull0 60.8 mm to (183.6, 104.5), turned to -90 degrees
- moved D4 53.9 mm to (187.8, 126.9), turned to 180 degrees
- moved Rled12 49.4 mm to (188.4, 130.7), turned to 0 degrees
- moved TP7 30.6 mm to (171.6, 81.5)
- moved Rled5 29.6 mm to (210.4, 126.2), turned to 180 degrees
- moved Cdec0 18.1 mm to (216.7, 128.7), turned to 180 degrees
- moved D5 9.69 mm to (209.0, 120.4), turned to 90 degrees
- moved Cfilt1 9.36 mm to (195.3, 88.8), turned to 180 degrees
- moved Cdec1 8.84 mm to (211.3, 120.9), turned to -90 degrees
- moved Cdec2 7.64 mm to (210.9, 112.7), turned to 90 degrees
- moved Cfilt2 4.79 mm to (203.2, 92.7)
- moved U4 4.66 mm to (216.7, 118.9), turned to 0 degrees
- moved D6 2.94 mm to (171.7, 88.4)
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Connections:
- Cfilt1 pad 1: Net-(U5B-+) -> Net-(U5A-+)
- Cfilt2 pad 1: Net-(U5A-+) -> Net-(U5B-+)
- J3 pad 10: SPICLK -> SPICS
- J3 pad 11: SPITX -> SPIRX
- J3 pad 12: SPIRX -> SPITX
- J3 pad 9: SPICS -> SPICLK
- R18 pad 2: Net-(U5B-+) -> Net-(U5A-+)
- R19 pad 1: Net-(U5B-+) -> Net-(U5A-+)
- R20 pad 2: Net-(U5A-+) -> Net-(U5B-+)
- R21 pad 1: Net-(U5A-+) -> Net-(U5B-+)
- U5 pad 1: MEAS1 -> MEAS2
- U5 pad 2: MEAS2 -> MEAS1
- U6 pad J4_1: MEAS1 -> MEAS3
- U6 pad J4_6: MEAS3 -> MEAS1
Routing:
- net +3.3V: track 2.10 -> 86.2 mm, vias 40 -> 1
- net PWM1A: track 5.05 -> 59.2 mm
- net PWM1B: track 11.9 -> 60.5 mm
- net NEUT: track 16.1 -> 61.1 mm
- net PWM2A: track 10.2 -> 44.3 mm
- net +5V: track 27.3 -> 59.6 mm, vias 0 -> 80
- net PWM2B: track 15.4 -> 43.8 mm
- net Net-(U5C-+): track 25.5 -> 45.2 mm, vias 2 -> 1
- net Net-(U5A-+): track 43.3 -> 27.2 mm
- net Net-(U5B-+): track 10.4 -> 25.4 mm, vias 2 -> 1
- net SPICLK: track 0.00 -> 14.3 mm
- net MEAS3: track 15.3 -> 29.2 mm, vias 0 -> 1
- net SPIRX: track 0.00 -> 12.2 mm
- net MEAS2: track 15.4 -> 26.5 mm, vias 0 -> 1
- net PWM3A: track 14.7 -> 25.8 mm
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- added copper zone on B.Cu, net +5V

Commit message: drc passed, only pwr in missing
Parts:
- moved TP3 8.87 mm to (171.6, 107.0)
- moved TP1 4.81 mm to (171.6, 102.5)
- moved TP2 4.72 mm to (171.6, 98.0)
- moved R3 4.00 mm to (175.4, 77.2)
- moved R4 4.00 mm to (177.9, 77.2)
- moved Rpull1 2.34 mm to (187.0, 95.0)
- moved Rpull2 2.27 mm to (187.0, 92.7)
- moved CBOOT3 1.78 mm to (214.0, 64.5)
- moved Cd3 1.78 mm to (226.3, 67.7)
- moved Cdec6 1.78 mm to (226.3, 70.0)
- moved D3 1.78 mm to (214.0, 68.5)
- moved Q5 1.78 mm to (216.6, 58.3)
- moved Q6 1.78 mm to (224.8, 58.3)
- moved R10 1.78 mm to (220.3, 77.2)
- moved R11 1.78 mm to (215.8, 66.1)
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Connections:
- U6 pad J4_4: MEAS2 -> MEAS1
- U6 pad J4_6: MEAS1 -> MEAS2
Routing:
- net FASE2: track 30.5 -> 20.7 mm
- net PWM1B: track 60.5 -> 64.9 mm
- net FASE3: track 27.9 -> 31.9 mm
- net MEAS1: track 22.5 -> 26.4 mm
- net MEAS2: track 26.5 -> 22.7 mm
- net PWM1A: track 59.2 -> 62.9 mm
- net FASE1: track 31.0 -> 32.0 mm
- net Net-(U5A-+): track 27.2 -> 27.9 mm
- net PWM3A: track 25.8 -> 25.1 mm
- net Net-(U5C-+): track 45.2 -> 45.9 mm
- net GND: vias 232 -> 320
- net +12V: vias 331 -> 355

Commit message: vias
Parts:
- moved CPWR0 15.6 mm to (168.0, 119.6), turned to 90 degrees
- moved Cdec2 6.89 mm to (217.0, 109.5), turned to -90 degrees
- moved J1 0.73 mm to (170.5, 132.0), turned to -90 degrees
Routing:
- net +5V: track 59.6 -> 50.9 mm
- net GND: vias 320 -> 605
- net +12V: vias 355 -> 226
Other:
- board size 67.4 x 94.6 mm -> 79.4 x 95.6 mm

Commit message: should be done?
Parts:
- moved D4 15.8 mm to (172.1, 126.8)
- moved Rled12 13.1 mm to (175.6, 128.2), turned to 90 degrees
- moved MEAS2 5.07 mm to (166.9, 96.0)
- moved MEAS1 4.88 mm to (166.9, 101.0)
- moved MEAS3 4.74 mm to (166.9, 106.0)
- moved NEUT 4.60 mm to (167.0, 81.5)
- moved J3 2.93 mm to (233.4, 104.7)
- moved CPWR0 0.05 mm to (167.9, 119.6)
- renumbered TP1 to MEAS1, TP2 to MEAS2, TP3 to MEAS3, TP7 to NEUT
Routing:
- net +12V: track 0.00 -> 13.0 mm, vias 226 -> 258
- net GND: track 23.3 -> 12.0 mm, vias 605 -> 615
- net MEAS3: track 28.8 -> 34.4 mm
- net NEUT: track 61.1 -> 65.7 mm
- net MEAS1: track 26.4 -> 30.4 mm
- net MEAS2: track 22.7 -> 26.5 mm
- net PWM3B: track 25.5 -> 29.2 mm
- net PWM1A: track 62.9 -> 66.3 mm
- net SPICS: track 9.97 -> 13.1 mm
- net SPICLK: track 14.8 -> 17.7 mm
- net PWM1B: track 64.9 -> 67.9 mm
- net SPIRX: track 12.7 -> 15.6 mm
- net SPITX: track 9.11 -> 12.0 mm
- net PWM2A: track 44.8 -> 47.7 mm
- net PWM2B: track 44.2 -> 47.1 mm
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- removed copper zone on In2.Cu, net +3.3V
