File: hw/lse1_pcb/lse1_pcb.kicad_sch (KiCad schematic)
At the start: 80 parts, among them J1 PWR_IN, J11 TP_FASE2, J12 TP_FASE1, J13 TP_FASE3, M1 Motor_3pin, Q1 IRFR1205, Q2 IRFR1205, Q3 IRFR1205, Q4 IRFR1205, Q5 IRFR1205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

Commit message: sortida lse1
Parts:
- Cd1, Cd2, Cd3: value 47u -> 4.7u
- Cfilt1, Cfilt2, Cfilt3: value C -> 4.7n
- R13, R14, R15, R16, R17: value R -> 1k
- R18, R20, R22: value R -> 33k
- R19, R21, R23: value R -> 12k
Changed lines of the file:
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@@
 			)
 		)
-		(property "Value" "R"
+		(property "Value" "33k"
 			(at 233.172 170.688 90)
 			(effects
@@
 			)
 		)
-		(property "Value" "R"
+		(property "Value" "33k"
 			(at 233.172 202.438 90)
 			(effects
@@
 			)
 		)
-		(property "Value" "47u"
+		(property "Value" "4.7u"
 			(at 190.246 30.48 90)
 			(effects
@@
 		(on_board yes)
 		(dnp no)
-		(fields_autoplaced yes)
 		(property "Reference" "#PWR04"
 			(at 189.23 74.93 0)
@@
 			)
 		)
-		(property "Value" "47u"
+		(property "Value" "4.7u"
 			(at 187.706 173.99 90)
 			(effects
@@
 			)
 		)
-		(property "Value" "C"
+		(property "Value" "4.7n"
 			(at 245.364 143.51 90)
 			(effects
@@
 			)
 		)
-		(property "Value" "R"
+		(property "Value" "12k"
 			(at 236.982 178.562 90)
 			(effects
@@
 			)
 		)
-		(property "Value" "R"
+		(property "Value" "1k"
 			(at 275.082 45.212 90)
 			(effects
@@
 			)
 		)
-		(property "Value" "R"
+		(property "Value" "1k"
 			(at 264.668 51.562 90)
 			(effects
@@
 			)
 		)
-		(property "Value" "R"
+		(property "Value" "12k"
 			(at 236.982 210.312 90)
 			(effects
@@
 			)
 		)
-		(property "Value" "C"
+		(property "Value" "4.7n"
 			(at 245.364 176.53 90)
 			(effects
@@
 			)
 		)
-		(property "Value" "R"
+		(property "Value" "33k"
 			(at 233.172 137.668 90)
 			(effects
@@
 			)
 		)
-		(property "Value" "47u"
+		(property "Value" "4.7u"
 			(at 188.976 102.87 90)
 			(effects
@@
 			)
 		)
+		(property "Field5" ""
+			(at 185.42 102.87 90)
+			(effects
+				(font
+					(size 1.27 1.27)
+				)
+				(hide yes)
+			)
+		)
 		(pin "2"
 		)
@@
 			)
 		)
-		(property "Value" "R"
+		(property "Value" "1k"
 			(at 275.082 57.912 90)
 			(effects
@@
 			)
 		)
-		(property "Value" "R"
+		(property "Value" "1k"
 			(at 277.368 51.562 90)
 			(effects
@@
 			)
 		)
-		(property "Value" "R"
+		(property "Value" "1k"
 			(at 275.082 69.342 90)
 			(effects
@@
 			)
 		)
-		(property "Value" "C"
+		(property "Value" "4.7n"
 			(at 245.364 208.28 90)
 			(effects
@@
 			)
 		)
-		(property "Value" "R"
+		(property "Value" "12k"
 			(at 236.982 145.542 90)
 			(effects

Commit message: PID v1, falla potenciometre
Parts:
- Cfilt1: value 4.7n -> 30n
Changed lines of the file:
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@@
 			)
 		)
-		(property "Value" "4.7n"
+		(property "Value" "30n"
 			(at 245.364 143.51 90)
 			(effects

Commit message: primer esbos SPI
Parts:
- CBOOT1: value C -> 100n
Changed lines of the file:
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@@
 			)
 		)
-		(property "Value" "C"
+		(property "Value" "100n"
 			(at 165.1 53.086 90)
 			(effects

Commit message: codi LSE1 retocat + motors calibrats
Parts:
- Cfilt2, Cfilt3: value 4.7n -> 30n
- R1, R11, R12, R2, R7, R8: value R -> 100
- R10, R3, R4, R5, R6, R9: value R -> 33
- R16: value 1k -> 33k
- R17: value 1k -> 15k
- R19, R21, R23: value 12k -> 15k
- Rpull1, Rpull2, Rpull3: value R -> 1k
Changed lines of the file:
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@@
 			)
 		)
-		(property "Value" "R"
+		(property "Value" "100"
 			(at 173.99 139.192 90)
 			(effects
@@
 			)
 		)
-		(property "Value" "R"
+		(property "Value" "1k"
 			(at 279.4 172.72 90)
 			(effects
@@
 			)
 		)
-		(property "Value" "R"
+		(property "Value" "100"
 			(at 175.26 66.802 90)
 			(effects
@@
 			)
 		)
-		(property "Value" "R"
+		(property "Value" "33"
 			(at 134.112 134.366 90)
 			(effects
@@
 			)
 		)
-		(property "Value" "R"
+		(property "Value" "33"
 			(at 132.842 204.216 90)
 			(effects
@@
 			)
 		)
-		(property "Value" "12k"
+		(property "Value" "15k"
 			(at 236.982 178.562 90)
 			(effects
@@
 			)
 		)
-		(property "Value" "R"
+		(property "Value" "33"
 			(at 132.842 194.818 90)
 			(effects
@@
 			)
 		)
-		(property "Value" "12k"
+		(property "Value" "15k"
 			(at 236.982 210.312 90)
 			(effects
@@
 			)
 		)
-		(property "Value" "R"
+		(property "Value" "33"
 			(at 134.112 124.968 90)
 			(effects
@@
 			)
 		)
-		(property "Value" "R"
+		(property "Value" "100"
 			(at 173.99 129.032 90)
 			(effects
@@
 			)
 		)
-		(property "Value" "R"
+		(property "Value" "33"
 			(at 135.382 52.578 90)
 			(effects
@@
 			)
 		)
-		(property "Value" "4.7n"
+		(property "Value" "30n"
 			(at 245.364 176.53 90)
 			(effects
@@
 			)
 		)
-		(property "Value" "R"
+		(property "Value" "100"
 			(at 172.72 198.882 90)
 			(effects
@@
 			)
 		)
-		(property "Value" "R"
+		(property "Value" "1k"
 			(at 279.4 139.7 90)
 			(effects
@@
 			)
 		)
-		(property "Value" "1k"
+		(property "Value" "33k"
 			(at 275.082 57.912 90)
 			(effects
@@
 			)
 		)
-		(property "Value" "R"
+		(property "Value" "1k"
 			(at 279.4 204.47 90)
 			(effects
@@
 			)
 		)
-		(property "Value" "R"
+		(property "Value" "100"
 			(at 175.26 56.642 90)
 			(effects
@@
 			)
 		)
-		(property "Value" "R"
+		(property "Value" "33"
 			(at 135.382 61.976 90)
 			(effects
@@
 			)
 		)
-		(property "Value" "R"
+		(property "Value" "100"
 			(at 172.72 209.042 90)
 			(effects
@@
 			)
 		)
-		(property "Value" "1k"
+		(property "Value" "15k"
 			(at 275.082 69.342 90)
 			(effects
@@
 			)
 		)
-		(property "Value" "4.7n"
+		(property "Value" "30n"
 			(at 245.364 208.28 90)
 			(effects
@@
 			)
 		)
-		(property "Value" "12k"
+		(property "Value" "15k"
 			(at 236.982 145.542 90)
 			(effects
