File: hw/lse1_pcb/_autosave-lse1_pcb.kicad_sch (KiCad schematic)
At the start: 80 parts, among them J1 PWR_IN, J11 TP_FASE2, J12 TP_FASE1, J13 TP_FASE3, M1 Motor_3pin, Q1 IRFR1205, Q2 IRFR1205, Q3 IRFR1205, Q4 IRFR1205, Q5 IRFR1205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

Commit message: update silkscreen
Parts:
- renumbered DATAOUT to DATAOUT1, NEUT to NEUT1, TP_MEAS to TP_MEAS1
Changed lines of the file:
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@@
 		(dnp no)
 		(fields_autoplaced yes)
-		(property "Reference" "DATAOUT"
+		(property "Reference" "DATAOUT1"
 			(at 58.42 194.31 0)
 			(effects
@@
 			(project ""
 				(path "/adaa4865-6386-49a6-8ca3-a43f702611f6"
-					(reference "DATAOUT")
+					(reference "DATAOUT1")
 					(unit 1)
 				)
@@
 		(dnp no)
 		(fields_autoplaced yes)
-		(property "Reference" "TP_MEAS"
+		(property "Reference" "TP_MEAS1"
 			(at 283.21 102.87 0)
 			(effects
@@
 			(project ""
 				(path "/adaa4865-6386-49a6-8ca3-a43f702611f6"
-					(reference "TP_MEAS")
+					(reference "TP_MEAS1")
 					(unit 1)
 				)
@@
 		(dnp no)
 		(fields_autoplaced yes)
-		(property "Reference" "NEUT"
+		(property "Reference" "NEUT1"
 			(at 292.1 68.5799 0)
 			(effects
@@
 			(project "lse1_pcb"
 				(path "/adaa4865-6386-49a6-8ca3-a43f702611f6"
-					(reference "NEUT")
+					(reference "NEUT1")
 					(unit 1)
 				)
